Commit message: update navigation

File: urdf/sim1.urdf (robot description, URDF)
Before this commit: robot my_robot, 8 links, 7 joints
Links:
- added link imu_link, mass 0.01; collision box size=0.02 0.02 0.01; visual box size=0.02 0.02 0.01
Joints:
- added joint imu_joint: type fixed, parent chassis, child imu_link, origin xyz=0 0 0.05 rpy=0 0 0

File: urdf/sim_copy.urdf (robot description, URDF)
Before this commit: robot my_robot, 8 links, 7 joints
Links:
- added link imu_link, mass 0.01; collision box size=0.02 0.02 0.01; visual box size=0.02 0.02 0.01
Joints:
- added joint imu_joint: type fixed, parent chassis, child imu_link, origin xyz=0 0 0.05 rpy=0 0 0
