Commit message: update all

File: urdf/sim.urdf (robot description, URDF)
Before this commit: robot my_robot, 8 links, 7 joints
Links:
- added link camera_link; collision box size=0.035 0.096 0.031; visual box size=0.024 0.094 0.029
- added link camera_optical_link
- added link imu_link, mass 0.01; collision box size=0.02 0.02 0.01; visual box size=0.02 0.02 0.01
Joints:
- added joint camera_joint: type fixed, parent chassis, child camera_link, origin xyz=0.1045 0 0.1055 rpy=0 0 0
- added joint camera_optical_joint: type fixed, parent camera_link, child camera_optical_link, origin xyz=0 0 0 rpy=-1.57079632679 0 -1.57079632679
- added joint imu_joint: type fixed, parent chassis, child imu_link, origin xyz=0 0 0.05 rpy=0 0 0

File: urdf/sim1.urdf (robot description, URDF)
Before this commit: robot my_robot, 9 links, 8 joints
Links:
- added link camera_link, mass 0.15; collision box size=0.035 0.096 0.031; visual box size=0.024 0.094 0.029
- added link camera_optical_link
- link chassis: mass 2.15 -> 4.4
- link left_front_wheel: mass 0.035 -> 0.1
- link left_rear_wheel: mass 0.035 -> 0.1
- link right_front_wheel: mass 0.035 -> 0.1
- link right_rear_wheel: mass 0.035 -> 0.1
Joints:
- added joint camera_joint: type fixed, parent chassis, child camera_link, origin xyz=0.1045 0 0.1055 rpy=0 0 0
- added joint camera_optical_joint: type fixed, parent camera_link, child camera_optical_link, origin xyz=0 0 0 rpy=-1.57079632679 0 -1.57079632679
